File: Eagle/USB-UART Bridge/UsbUartBridge.sch (EAGLE design)
At the start: 7 parts, among them IC1 CP210X_USB_UART, X1 USB-A-H

Commit message: finalized schematic design
Parts:
- removed JP2: (no value), SparkFun:M07
- added JP1: (no value), SparkFun:M06SIP
Connections:
- removed net CTS: IC1.CTS, JP2.2
- removed net RST: JP2.6
- removed net RTS: IC1.RTS
- new net DTR: IC1.DTR, JP1.6
- net 3V3: no longer JP2.7
- net 5V: now also JP1.3; no longer JP2.3
- net GND: now also JP1.1, JP1.2; no longer JP2.1
- net RXD: now also JP1.5; no longer JP2.5
- net TXD: now also JP1.4; no longer JP2.4
Changed lines of the file:
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@@
 <part name="R1" library="rcl" deviceset="R-EU_" device="0204/7" value="330"/>
 <part name="LED1" library="adafruit" deviceset="LED" device="3MM"/>
-<part name="JP2" library="SparkFun" deviceset="M07" device=""/>
+<part name="JP1" library="SparkFun" deviceset="M06" device="SIP"/>
 </parts>
 <sheets>
@@
 <instance part="R1" gate="G$1" x="68.58" y="83.82"/>
 <instance part="LED1" gate="G$1" x="76.2" y="83.82" rot="R90"/>
-<instance part="JP2" gate="G$1" x="175.26" y="116.84" rot="R180"/>
+<instance part="JP1" gate="G$1" x="175.26" y="116.84" rot="R180"/>
 </instances>
 <busses>
@@
 </segment>
 <segment>
-<wire x1="160.02" y1="116.84" x2="170.18" y2="116.84" width="0.1524" layer="91"/>
-<pinref part="JP2" gate="G$1" pin="3"/>
-<label x="160.02" y="116.84" size="1.778" layer="95"/>
+<pinref part="JP1" gate="G$1" pin="3"/>
+<wire x1="162.56" y1="116.84" x2="170.18" y2="116.84" width="0.1524" layer="91"/>
+<label x="162.56" y="116.84" size="1.778" layer="95"/>
 </segment>
 </net>
@@
 </segment>
 <segment>
-<wire x1="160.02" y1="121.92" x2="170.18" y2="121.92" width="0.1524" layer="91"/>
-<pinref part="JP2" gate="G$1" pin="1"/>
-<label x="160.02" y="121.92" size="1.778" layer="95"/>
+<pinref part="JP1" gate="G$1" pin="1"/>
+<wire x1="162.56" y1="121.92" x2="170.18" y2="121.92" width="0.1524" layer="91"/>
+<label x="162.56" y="121.92" size="1.778" layer="95"/>
+</segment>
+<segment>
+<pinref part="JP1" gate="G$1" pin="2"/>
+<wire x1="162.56" y1="119.38" x2="170.18" y2="119.38" width="0.1524" layer="91"/>
+<label x="162.56" y="119.38" size="1.778" layer="95"/>
 </segment>
 </net>
@@
 <label x="73.66" y="104.14" size="1.778" layer="95"/>
 </segment>
-<segment>
-<pinref part="JP2" gate="G$1" pin="7"/>
-<wire x1="160.02" y1="106.68" x2="170.18" y2="106.68" width="0.1524" layer="91"/>
-<label x="160.02" y="106.68" size="1.778" layer="95"/>
-</segment>
-</net>
-<net name="RTS" class="0">
-<segment>
-<pinref part="IC1" gate="G$1" pin="RTS"/>
-<wire x1="149.86" y1="99.06" x2="139.7" y2="99.06" width="0.1524" layer="91"/>
-<label x="147.32" y="99.06" size="1.778" layer="95"/>
-</segment>
-</net>
-<net name="CTS" class="0">
-<segment>
-<pinref part="IC1" gate="G$1" pin="CTS"/>
-<wire x1="149.86" y1="96.52" x2="139.7" y2="96.52" width="0.1524" layer="91"/>
-<label x="147.32" y="96.52" size="1.778" layer="95"/>
-</segment>
-<segment>
-<wire x1="160.02" y1="119.38" x2="170.18" y2="119.38" width="0.1524" layer="91"/>
-<pinref part="JP2" gate="G$1" pin="2"/>
-<label x="160.02" y="119.38" size="1.778" layer="95"/>
-</segment>
 </net>
 <net name="RXD" class="0">
@@
 </segment>
 <segment>
-<wire x1="160.02" y1="111.76" x2="170.18" y2="111.76" width="0.1524" layer="91"/>
-<pinref part="JP2" gate="G$1" pin="5"/>
-<label x="160.02" y="111.76" size="1.778" layer="95"/>
+<pinref part="JP1" gate="G$1" pin="5"/>
+<wire x1="162.56" y1="111.76" x2="170.18" y2="111.76" width="0.1524" layer="91"/>
+<label x="162.56" y="111.76" size="1.778" layer="95"/>
 </segment>
 </net>
@@
 </segment>
 <segment>
-<wire x1="160.02" y1="114.3" x2="170.18" y2="114.3" width="0.1524" layer="91"/>
-<pinref part="JP2" gate="G$1" pin="4"/>
-<label x="160.02" y="114.3" size="1.778" layer="95"/>
+<pinref part="JP1" gate="G$1" pin="4"/>
+<wire x1="162.56" y1="114.3" x2="170.18" y2="114.3" width="0.1524" layer="91"/>
+<label x="162.56" y="114.3" size="1.778" layer="95"/>
 </segment>
 </net>
-<net name="RST" class="0">
+<net name="DTR" class="0">
 <segment>
-<wire x1="160.02" y1="109.22" x2="170.18" y2="109.22" width="0.1524" layer="91"/>
-<pinref part="JP2" gate="G$1" pin="6"/>
-<label x="160.02" y="109.22" size="1.778" layer="95"/>
+<pinref part="IC1" gate="G$1" pin="DTR"/>
+<wire x1="149.86" y1="109.22" x2="139.7" y2="109.22" width="0.1524" layer="91"/>
+<label x="147.32" y="109.22" size="1.778" layer="95"/>
+</segment>
+<segment>
+<pinref part="JP1" gate="G$1" pin="6"/>
+<wire x1="162.56" y1="109.22" x2="170.18" y2="109.22" width="0.1524" layer="91"/>
+<label x="162.56" y="109.22" size="1.778" layer="95"/>
 </segment>
 </net>
